File: kicad/big_battery/big_battery.kicad_pcb (KiCad board)
At the start: 2 copper layers, 35 x 35 mm, 31 parts, among them J1 CN2, J2 CN3, J3 MCU, Q1 AO3400, U1 AP1117-ADJ, U2 LMV324

Commit message: pretty much working board, requires some bodges on the op-amp and extra potentiometers
Parts:
- C2: value C_Small -> 0.1uF
- C6, C7: value NC -> 0.1uF
- L1: value L_Small -> JUMPER
- R1: value R_Small -> 13K 1%
- R10: value R_Small -> 100K
- R11: value R_Small -> 3.3K 1%
- R12: value R_Small -> 3.9K 1%
- R13, R15, R2, R5: value R_Small -> 10K 1%
- R16: value R_Small -> 12K 1%
- R3: value 500K -> 500K 1%
- R4: value R_Small -> 180K 1%
- R6: value R_Small -> 4.7K 1%
- R7: value R_Small -> 16K 1%
- R8: value 10K -> 10K 1%
- R9: value R_Small -> 1K
Connections:
- R10 pad 1: Net-(Q1-Pad1) -> GND
- R10 pad 2: +3V3 -> Net-(Q1-Pad1)
Changed lines of the file:
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@@
-(kicad_pcb (version 20171130) (host pcbnew 5.0.1-33cea8e~67~ubuntu18.04.1)
+(kicad_pcb (version 20171130) (host pcbnew 5.0.1-33cea8e~68~ubuntu18.04.1)
   (general
     (thickness 1.6)
@@
       (effects (font (size 1 1) (thickness 0.15)))
     )
-    (fp_text value NC (at 0 1.43) (layer F.Fab)
+    (fp_text value 0.1uF (at 0 1.43) (layer F.Fab)
       (effects (font (size 1 1) (thickness 0.15)))
     )
@@
       (effects (font (size 1 1) (thickness 0.15)))
     )
-    (fp_text value C_Small (at 0 1.43) (layer F.Fab)
+    (fp_text value 0.1uF (at 0 1.43) (layer F.Fab)
       (effects (font (size 1 1) (thickness 0.15)))
     )
@@
       (effects (font (size 1 1) (thickness 0.15)))
     )
-    (fp_text value NC (at 0 1.43 90) (layer F.Fab)
+    (fp_text value 0.1uF (at 0 1.43 90) (layer F.Fab)
       (effects (font (size 1 1) (thickness 0.15)))
     )
@@
       (effects (font (size 1 1) (thickness 0.15)))
     )
-    (fp_text value L_Small (at 0 1.43 180) (layer F.Fab)
+    (fp_text value JUMPER (at 0 1.43 180) (layer F.Fab)
       (effects (font (size 1 1) (thickness 0.15)))
     )
@@
       (effects (font (size 1 1) (thickness 0.15)))
     )
-    (fp_text value 10K (at 0 1.43 270) (layer F.Fab)
+    (fp_text value "10K 1%" (at 0 1.43 270) (layer F.Fab)
       (effects (font (size 1 1) (thickness 0.15)))
     )
@@
       (effects (font (size 1 1) (thickness 0.15)))
     )
-    (fp_text value R_Small (at 0 1.43 270) (layer F.Fab)
+    (fp_text value 1K (at 0 1.43 270) (layer F.Fab)
       (effects (font (size 1 1) (thickness 0.15)))
     )
@@
       (effects (font (size 1 1) (thickness 0.15)))
     )
-    (fp_text value R_Small (at 0 1.43) (layer F.Fab)
+    (fp_text value "10K 1%" (at 0 1.43) (layer F.Fab)
       (effects (font (size 1 1) (thickness 0.15)))
     )
@@
       (effects (font (size 1 1) (thickness 0.15)))
     )
-    (fp_text value R_Small (at 0 1.43 270) (layer F.Fab)
+    (fp_text value "180K 1%" (at 0 1.43 270) (layer F.Fab)
       (effects (font (size 1 1) (thickness 0.15)))
     )
@@
       (effects (font (size 1 1) (thickness 0.15)))
     )
-    (fp_text value 500K (at 0 1.43 180) (layer F.Fab)
+    (fp_text value "500K 1%" (at 0 1.43 180) (layer F.Fab)
       (effects (font (size 1 1) (thickness 0.15)))
     )
@@
       (effects (font (size 1 1) (thickness 0.15)))
     )
-    (fp_text value R_Small (at 0 1.43 180) (layer F.Fab)
+    (fp_text value "10K 1%" (at 0 1.43 180) (layer F.Fab)
       (effects (font (size 1 1) (thickness 0.15)))
     )
@@
       (effects (font (size 1 1) (thickness 0.15)))
     )
-    (fp_text value R_Small (at 0 1.43 180) (layer F.Fab)
+    (fp_text value "13K 1%" (at 0 1.43 180) (layer F.Fab)
       (effects (font (size 1 1) (thickness 0.15)))
     )
@@
       (effects (font (size 1 1) (thickness 0.15)))
     )
-    (fp_text value R_Small (at 0 1.43 270) (layer F.Fab)
+    (fp_text value "16K 1%" (at 0 1.43 270) (layer F.Fab)
       (effects (font (size 1 1) (thickness 0.15)))
     )
@@
       (effects (font (size 1 1) (thickness 0.15)))
     )
-    (fp_text value R_Small (at 0 1.43 90) (layer F.Fab)
+    (fp_text value 100K (at 0 1.43 90) (layer F.Fab)
       (effects (font (size 1 1) (thickness 0.15)))
     )
@@
     (fp_line (start -0.8 0.4) (end -0.8 -0.4) (layer F.Fab) (width 0.1))
     (pad 2 smd roundrect (at 0.875 0 90) (size 1.05 0.95) (layers F.Cu F.Paste F.Mask) (roundrect_rratio 0.25)
-      (net 5 +3V3))
+      (net 10 "Net-(Q1-Pad1)"))
     (pad 1 smd roundrect (at -0.875 0 90) (size 1.05 0.95) (layers F.Cu F.Paste F.Mask) (roundrect_rratio 0.25)
-      (net 10 "Net-(Q1-Pad1)"))
+      (net 3 GND))
     (model ${KISYS3DMOD}/Resistor_SMD.3dshapes/R_0603_1608Metric.wrl
       (at (xyz 0 0 0))
@@
       (effects (font (size 1 1) (thickness 0.15)))
     )
-    (fp_text value R_Small (at 0 1.43 180) (layer F.Fab)
+    (fp_text value "3.3K 1%" (at 0 1.43 180) (layer F.Fab)
       (effects (font (size 1 1) (thickness 0.15)))
     )
@@
       (effects (font (size 1 1) (thickness 0.15)))
     )
-    (fp_text value R_Small (at 0 1.43 270) (layer F.Fab)
+    (fp_text value "3.9K 1%" (at 0 1.43 270) (layer F.Fab)
       (effects (font (size 1 1) (thickness 0.15)))
     )
@@
       (effects (font (size 1 1) (thickness 0.15)))
     )
-    (fp_text value R_Small (at 0 1.43 270) (layer F.Fab)
+    (fp_text value "10K 1%" (at 0 1.43 270) (layer F.Fab)
       (effects (font (size 1 1) (thickness 0.15)))
     )
@@
       (effects (font (size 1 1) (thickness 0.15)))
     )
-    (fp_text value R_Small (at 0 1.43 90) (layer F.Fab)
+    (fp_text value "10K 1%" (at 0 1.43 90) (layer F.Fab)
       (effects (font (size 1 1) (thickness 0.15)))
     )
@@
       (effects (font (size 1 1) (thickness 0.15)))
     )
-    (fp_text value R_Small (at 0 1.43 90) (layer F.Fab)
+    (fp_text value "12K 1%" (at 0 1.43 90) (layer F.Fab)
       (effects (font (size 1 1) (thickness 0.15)))
     )
@@
       (effects (font (size 1 1) (thickness 0.15)))
     )
-    (fp_text value R_Small (at 0 1.43 180) (layer F.Fab)
-      (effects (font (size 1 1) (thickness 0.15)))
-    )
+    (fp_text value "4.7K 1%" (at 0 1.43 180) (layer F.Fab)
+      (effects (font (size 1 1) (thickness 0.15)))
+    )
