File: kicad/big_battery/big_battery.sch (KiCad schematic (older format))
At the start: 31 parts, among them J1 CN2, J2 CN3, Q1 AO3400, U1 AP1117-ADJ, U2 LMV324

Commit message: fixes component selection script
Parts:
- added D?: LED_Small, symbol Device:LED_Small
- added R?: 100K, Resistor_SMD:R_0603_1608Metric_Pad1.05x0.95mm_HandSolder, symbol Device:R_Small
- R1: value R_Small -> 13K 1%
- R10: value R_Small -> 100K
- R11: value R_Small -> 3.3K 1%
- R12: value R_Small -> 3.9K 1%
- R13, R2, R5: value R_Small -> 10K 1%
- R3: value 500K -> 5M 1%
- R4: value R_Small -> 1.8M 1%
- R6: value R_Small -> 4.7K 1%
- R7: value R_Small -> 16K 1%
- R8: value 10K -> 10K 1%
- R9: value R_Small -> 1K
Connections:
- wire segments 127 -> 135
Other:
- note added: "#Global Setting\nV_adc_max = 2.4 #Max voltage the ADC can read\nADC_resolution = 4096 #Resolution of ADC\n\nV_op = 3.3 #Supply voltage of OP-AMPs and analog circuitry, sets LDO output voltage\n\n\nV_max = 5.5 #Max voltage of Power supply\nI_max = 120 #Max amperage of the Power supply\n\nI_over_current = 10 #Over current set point (amps)\nI_trickle_current = 1 #Trickle current set point (amps)\n\n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"
- moved on the sheet: Q1, R10, R9
Changed lines of the file:
@@
 	3350 1000 3500 1000
 Wire Wire Line
-	3950 1000 3950 1100
+	3950 1000 3950 1050
 $Comp
 L Device:R_Small R7
@@
 P 3500 1200
 F 0 "R7" H 3559 1246 50  0000 L CNN
-F 1 "R_Small" H 3559 1155 50  0000 L CNN
+F 1 "16K 1%" H 3559 1155 50  0000 L CNN
 F 2 "Resistor_SMD:R_0603_1608Metric_Pad1.05x0.95mm_HandSolder" H 3500 1200 50  0001 C CNN
 F 3 "~" H 3500 1200 50  0001 C CNN
@@
 P 3500 1600
 F 0 "R8" H 3559 1646 50  0000 L CNN
-F 1 "10K" H 3559 1555 50  0000 L CNN
+F 1 "10K 1%" H 3559 1555 50  0000 L CNN
 F 2 "Resistor_SMD:R_0603_1608Metric_Pad1.05x0.95mm_HandSolder" H 3500 1600 50  0001 C CNN
 F 3 "~" H 3500 1600 50  0001 C CNN
@@
 $EndComp
 Wire Wire Line
-	3950 1750 3950 1300
+	3950 1750 3950 1650
 Wire Wire Line
 	3500 1700 3500 1750
@@
 P 2300 5200
 F 0 "R3" V 2104 5200 50  0000 C CNN
-F 1 "500K" V 2195 5200 50  0000 C CNN
+F 1 "5M 1%" V 2195 5200 50  0000 C CNN
 F 2 "Resistor_SMD:R_0603_1608Metric_Pad1.05x0.95mm_HandSolder" H 2300 5200 50  0001 C CNN
 F 3 "~" H 2300 5200 50  0001 C CNN
@@
 P 2650 4850
 F 0 "R4" H 2591 4804 50  0000 R CNN
-F 1 "R_Small" H 2591 4895 50  0000 R CNN
+F 1 "1.8M 1%" H 2591 4895 50  0000 R CNN
 F 2 "Resistor_SMD:R_0603_1608Metric_Pad1.05x0.95mm_HandSolder" H 2650 4850 50  0001 C CNN
 F 3 "~" H 2650 4850 50  0001 C CNN
@@
 P 3100 6150
 F 0 "R6" V 3296 6150 50  0000 C CNN
-F 1 "R_Small" V 3205 6150 50  0000 C CNN
+F 1 "4.7K 1%" V 3205 6150 50  0000 C CNN
 F 2 "Resistor_SMD:R_0603_1608Metric_Pad1.05x0.95mm_HandSolder" H 3100 6150 50  0001 C CNN
 F 3 "~" H 3100 6150 50  0001 C CNN
@@
 P 2650 6750
 F 0 "R5" H 2709 6796 50  0000 L CNN
-F 1 "R_Small" H 2709 6705 50  0000 L CNN
+F 1 "10K 1%" H 2709 6705 50  0000 L CNN
 F 2 "Resistor_SMD:R_0603_1608Metric_Pad1.05x0.95mm_HandSolder" H 2650 6750 50  0001 C CNN
 F 3 "~" H 2650 6750 50  0001 C CNN
@@
 P 6550 5650
 F 0 "R13" H 6491 5696 50  0000 R CNN
-F 1 "R_Small" H 6491 5605 50  0000 R CNN
+F 1 "10K 1%" H 6491 5605 50  0000 R CNN
 F 2 "Resistor_SMD:R_0603_1608Metric_Pad1.05x0.95mm_HandSolder" H 6550 5650 50  0001 C CNN
 F 3 "~" H 6550 5650 50  0001 C CNN
@@
 P 5950 5650
 F 0 "R11" H 5891 5604 50  0000 R CNN
-F 1 "R_Small" H 5891 5695 50  0000 R CNN
+F 1 "3.3K 1%" H 5891 5695 50  0000 R CNN
 F 2 "Resistor_SMD:R_0603_1608Metric_Pad1.05x0.95mm_HandSolder" H 5950 5650 50  0001 C CNN
 F 3 "~" H 5950 5650 50  0001 C CNN
@@
 L Device:Q_NMOS_GSD Q1
 U 1 1 5BCFF343
-P 5850 6150
-F 0 "Q1" H 6055 6196 50  0000 L CNN
-F 1 "AO3400" H 6055 6105 50  0000 L CNN
-F 2 "Package_TO_SOT_SMD:SOT-23_Handsoldering" H 6050 6250 50  0001 C CNN
-F 3 "~" H 5850 6150 50  0001 C CNN
-	1    5850 6150
+P 5850 6050
+F 0 "Q1" H 6055 6096 50  0000 L CNN
+F 1 "AO3400" H 6055 6005 50  0000 L CNN
+F 2 "Package_TO_SOT_SMD:SOT-23_Handsoldering" H 6050 6150 50  0001 C CNN
+F 3 "~" H 5850 6050 50  0001 C CNN
+	1    5850 6050
 	1    0    0    -1
 $EndComp
@@
 L Device:R_Small R10
 U 1 1 5BCFF619
-P 5400 5750
-F 0 "R10" H 5341 5704 50  0000 R CNN
-F 1 "R_Small" H 5341 5795 50  0000 R CNN
-F 2 "Resistor_SMD:R_0603_1608Metric_Pad1.05x0.95mm_HandSolder" H 5400 5750 50  0001 C CNN
-F 3 "~" H 5400 5750 50  0001 C CNN
-	1    5400 5750
-	-1   0    0    1
+P 5500 6250
+F 0 "R10" H 5441 6204 50  0000 R CNN
+F 1 "100K" H 5441 6295 50  0000 R CNN
+F 2 "Resistor_SMD:R_0603_1608Metric_Pad1.05x0.95mm_HandSolder" H 5500 6250 50  0001 C CNN
+F 3 "~" H 5500 6250 50  0001 C CNN
+	1    5500 6250
+	1    0    0    1
 $EndComp
 $Comp
 L Device:R_Small R9
 U 1 1 5BCFF687
-P 5200 6150
-F 0 "R9" V 5396 6150 50  0000 C CNN
-F 1 "R_Small" V 5305 6150 50  0000 C CNN
-F 2 "Resistor_SMD:R_0603_1608Metric_Pad1.05x0.95mm_HandSolder" H 5200 6150 50  0001 C CNN
-F 3 "~" H 5200 6150 50  0001 C CNN
-	1    5200 6150
+P 5200 6050
+F 0 "R9" V 5396 6050 50  0000 C CNN
+F 1 "1K" V 5305 6050 50  0000 C CNN
+F 2 "Resistor_SMD:R_0603_1608Metric_Pad1.05x0.95mm_HandSolder" H 5200 6050 50  0001 C CNN
+F 3 "~" H 5200 6050 50  0001 C CNN
+	1    5200 6050
 	0    -1   -1   0
 $EndComp
@@
 P 6250 4450
 F 0 "R12" H 6191 4404 50  0000 R CNN
-F 1 "R_Small" H 6191 4495 50  0000 R CNN
+F 1 "3.9K 1%" H 6191 4495 50  0000 R CNN
 F 2 "Resistor_SMD:R_0603_1608Metric_Pad1.05x0.95mm_HandSolder" H 6250 4450 50  0001 C CNN
 F 3 "~" H 6250 4450 50  0001 C CNN
@@
 	7450 4550 7700 4550
 Wire Wire Line
-	5950 5750 5950 5950
+	5950 5750 5950 5850
 Wire Wire Line
 	6550 5750 6550 6500
@@
 	6550 6500 6250 6500
 Wire Wire Line
-	5950 6500 5950 6350
+	5950 6500 5950 6250
 $Comp
 L power:GND #PWR015
@@
 Wire Wire Line
 	6250 6500 5950 6500
-Wire Wire Line
-	5400 5850 5400 6150
-Wire Wire Line
-	5400 6150 5300 6150
-Wire Wire Line
-	5400 6150 5650 6150
-Connection ~ 5400 6150
 $Comp
 L power:+3V3 #PWR014
@@
 Wire Wire Line
 	6250 4300 6250 4350
-$Comp
-L power:+3V3 #PWR013
-U 1 1 5BD0E62E
-P 5400 5600
-F 0 "#PWR013" H 5400 5450 50  0001 C CNN
-F 1 "+3V3" H 5415 5773 50  0000 C CNN
-F 2 "" H 5400 5600 50  0001 C CNN
-F 3 "" H 5400 5600 50  0001 C CNN
-	1    5400 5600
-	1    0    0    -1
-$EndComp
-Wire Wire Line
-	5400 5600 5400 5650
-Text Label 4850 6150 2    50   ~ 0
+Text Label 4850 6050 2    50   ~ 0
 TRICKLE_DIS
 $Comp
@@
 P 2250 3250
 F 0 "R2" H 2191 3204 50  0000 R CNN
-F 1 "R_Small" H 2191 3295 50  0000 R CNN
+F 1 "10K 1%" H 2191 3295 50  0000 R CNN
 F 2 "Resistor_SMD:R_0603_1608Metric_Pad1.05x0.95mm_HandSolder" H 2250 3250 50  0001 C CNN
 F 3 "~" H 2250 3250 50  0001 C CNN
@@
 P 2250 2750
 F 0 "R1" H 2191 2704 50  0000 R CNN
-F 1 "R_Small" H 2191 2795 50  0000 R CNN
+F 1 "13K 1%" H 2191 2795 50  0000 R CNN
 F 2 "Resistor_SMD:R_0603_1608Metric_Pad1.05x0.95mm_HandSolder" H 2250 2750 50  0001 C CNN
 F 3 "~" H 2250 2750 50  0001 C CNN
@@
 VOLTAGE TRM ADJ BETWEEN 0-2.5V
 Wire Wire Line
-	4900 6150 4900 3300
+	4900 6050 4900 3300
 Wire Wire Line
 	4900 3300 10400 3300
-Connection ~ 4900 6150
-Wire Wire Line
-	4900 6150 4850 6150
+Connection ~ 4900 6050
+Wire Wire Line
+	4900 6050 4850 6050
 Wire Wire Line
 	4800 5300 4800 3200
@@
 	2250 3450 2250 3350
 Wire Wire Line
-	4900 6150 5100 6150
+	4900 6050 5100 6050
 $Comp
 L Connector:Conn_01x04_Female J?
@@
 Text Label 10400 3300 2    50   ~ 0
 TRICKLE_DIS
+Wire Wire Line
+	5300 6050 5500 6050
+Wire Wire Line
+	5950 6500 5500 6500
+Wire Wire Line
+	5500 6500 5500 6350
+Connection ~ 5950 6500
+Wire Wire Line
+	5500 6150 5500 6050
+Connection ~ 5500 6050
+Wire Wire Line
+	5500 6050 5650 6050
+$Comp
+L Device:LED_Small D?
+U 1 1 5BD9A687
+P 4450 1500
+F 0 "D?" V 4496 1432 50  0000 R CNN
+F 1 "LED_Small" V 4405 1432 50  0000 R CNN
+F 2 "" V 4450 1500 50  0001 C CNN
+F 3 "~" V 4450 1500 50  0001 C CNN
+	1    4450 1500
+	0    -1   -1   0
+$EndComp
+$Comp
+L Device:R_Small R?
+U 1 1 5BD9AD09
+P 4450 1250
+F 0 "R?" H 4509 1296 50  0000 L CNN
+F 1 "100K" H 4509 1205 50  0000 L CNN
+F 2 "Resistor_SMD:R_0603_1608Metric_Pad1.05x0.95mm_HandSolder" H 4450 1250 50  0001 C CNN
+F 3 "~" H 4450 1250 50  0001 C CNN
+	1    4450 1250
+	1    0    0    -1
+$EndComp
+Wire Wire Line
+	4450 1150 4450 1050
+Wire Wire Line
+	4450 1050 3950 1050
+Connection ~ 3950 1050
+Wire Wire Line
+	3950 1050 3950 1100
+Wire Wire Line
+	4450 1350 4450 1400
+Wire Wire Line
+	4450 1600 4450 1650
+Wire Wire Line
+	4450 1650 3950 1650
+Connection ~ 3950 1650
+Wire Wire Line
+	3950 1650 3950 1300
+Text Notes 0 0  0    50   ~ 0
+#Global Setting\nV_adc_max = 2.4 #Max voltage the ADC can read\nADC_resolution = 4096 #Resolution of ADC\n\nV_op = 3.3 #Supply voltage of OP-AMPs and analog circuitry, sets LDO output voltage\n\n\nV_max =  5.5 #Max voltage of Power supply\nI_max = 120 #Max amperage of the Power supply\n\nI_over_current = 10 #Over current set point (amps)\nI_trickle_current = 1 #Trickle current set point (amps)\n\nV_trm = 4.2 #Power supply volatage set point\n\n
 $EndSCHEMATC

Commit message: pretty much working board, requires some bodges on the op-amp and extra potentiometers
Parts:
- C1, C3, C4, C5: symbol Device:C_Small -> big_battery-rescue:C_Small-Device
- C2: value C_Small -> 0.1uF; symbol Device:C_Small -> big_battery-rescue:C_Small-Device
- C6, C7: value NC -> 0.1uF; symbol Device:C_Small -> big_battery-rescue:C_Small-Device
- D1: symbol Device:D_Schottky_Small -> big_battery-rescue:D_Schottky_Small-Device
- D2: renamed from D?; symbol Device:LED_Small -> big_battery-rescue:LED_Small-Device
- J1: symbol Connector:Conn_01x04_Female -> big_battery-rescue:Conn_01x04_Female-Connector
- J2: symbol Connector:Conn_01x02_Female -> big_battery-rescue:Conn_01x02_Female-Connector
- J3: renamed from J?; symbol Connector:Conn_01x04_Female -> big_battery-rescue:Conn_01x04_Female-Connector
- L1: symbol Device:L_Small -> big_battery-rescue:L_Small-Device
- Q1: symbol Device:Q_NMOS_GSD -> big_battery-rescue:Q_NMOS_GSD-Device
- R1, R10, R13, R14, R2, R5, R7, R8, R9: symbol Device:R_Small -> big_battery-rescue:R_Small-Device
- R11: value 3.3K 1% -> 18K 1%; symbol Device:R_Small -> big_battery-rescue:R_Small-Device
- R12: value 3.9K 1% -> 4.3K 1%; symbol Device:R_Small -> big_battery-rescue:R_Small-Device
- R15: value R_Small -> 10K 1%; symbol Device:R_Small -> big_battery-rescue:R_Small-Device
- R16: value R_Small -> 12K 1%; symbol Device:R_Small -> big_battery-rescue:R_Small-Device
- R17: renamed from R?; symbol Device:R_Small -> big_battery-rescue:R_Small-Device
- R3: value 5M 1% -> 500K 1%; symbol Device:R_Small -> big_battery-rescue:R_Small-Device
- R4: value 1.8M 1% -> 180K 1%; symbol Device:R_Small -> big_battery-rescue:R_Small-Device
- R6: value 4.7K 1% -> 1.8K 1%; symbol Device:R_Small -> big_battery-rescue:R_Small-Device
- U1: symbol Regulator_Linear:AP1117-ADJ -> big_battery-rescue:AP1117-ADJ-Regulator_Linear
- U2: symbol Amplifier_Operational:LMV324 -> big_battery-rescue:LMV324-Amplifier_Operational
Other:
- note added: "#Global Setting\nV_adc_max = 2.35 #Max voltage the ADC can read\nADC_resolution = 4096 #Resolution of ADC\n\nV_op = 3.3 #Supply voltage of OP-AMPs and analog circuitry, sets LDO output voltage\n\n\nV_max = 5.5 #Max voltage of Power supply\nI_max = 120 #Max amperage of the Power supply\n\nI_over_current = 50 #Over current set point (amps)\nI_trickle_current = 1 #Trickle current set point (amps)\n\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"
- note added: "2"
- note added: "6"
- note added: "7\n"
- note added: "8"
- note added: "ADD POT"
- note added: "NOTE: + and - on U2B are reversed/WRONG"
- note removed: "#Global Setting\nV_adc_max = 2.4 #Max voltage the ADC can read\nADC_resolution = 4096 #Resolution of ADC\n\nV_op = 3.3 #Supply voltage of OP-AMPs and analog circuitry, sets LDO output voltage\n\n\nV_max = 5.5 #Max voltage of Power supply\nI_max = 120 #Max amperage of the Power supply\n\nI_over_current = 10 #Over current set point (amps)\nI_trickle_current = 1 #Trickle current set point (amps)\n\n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"

Commit message: attempt to fix kicad symbol library
Parts:
- C1, C2, C3, C4, C5, C6, C7: symbol big_battery-rescue:C_Small-Device -> Device:C_Small
- D1: symbol big_battery-rescue:D_Schottky_Small-Device -> Device:D_Schottky_Small
- D2: symbol big_battery-rescue:LED_Small-Device -> Device:LED_Small
- J1, J3: symbol big_battery-rescue:Conn_01x04_Female-Connector -> Connector:Conn_01x04_Female
- J2: symbol big_battery-rescue:Conn_01x02_Female-Connector -> Connector:Conn_01x02_Female
- L1: symbol big_battery-rescue:L_Small-Device -> Device:L_Small
- Q1: symbol big_battery-rescue:Q_NMOS_GSD-Device -> Device:Q_NMOS_GSD
- R1, R10, R11, R12, R13, R14, R15, R16, R17, R2, R3, R4, R5, R6, R7, R8, R9: symbol big_battery-rescue:R_Small-Device -> Device:R_Small_US
- U1: symbol big_battery-rescue:AP1117-ADJ-Regulator_Linear -> Regulator_Linear:AP1117-ADJ
- U2: symbol big_battery-rescue:LMV324-Amplifier_Operational -> Amplifier_Operational:LM324
Changed lines of the file:
@@
 $EndDescr
 $Comp
-L big_battery-rescue:LMV324-Amplifier_Operational U2
+L Amplifier_Operational:LM324 U2
 U 1 1 5BCEB1BA
 P 3200 5300
@@
 $EndComp
 $Comp
-L big_battery-rescue:LMV324-Amplifier_Operational U2
+L Amplifier_Operational:LM324 U2
 U 2 1 5BCEB218
 P 7250 5200
@@
 $EndComp
 $Comp
-L big_battery-rescue:LMV324-Amplifier_Operational U2
+L Amplifier_Operational:LM324 U2
 U 3 1 5BCEB2D7
 P 9750 5250
@@
 $EndComp
 $Comp
-L big_battery-rescue:LMV324-Amplifier_Operational U2
+L Amplifier_Operational:LM324 U2
 U 4 1 5BCEB31B
 P 3150 3100
@@
 $EndComp
 $Comp
-L big_battery-rescue:LMV324-Amplifier_Operational U2
+L Amplifier_Operational:LM324 U2
 U 5 1 5BCEB382
 P 3200 5300
@@
 $EndComp
 $Comp
-L big_battery-rescue:C_Small-Device C3
+L Device:C_Small C3
 U 1 1 5BCEB613
 P 3400 4600
@@
 $EndComp
 $Comp
-L big_battery-rescue:L_Small-Device L1
+L Device:L_Small L1
 U 1 1 5BCEB8DE
 P 2900 4450
@@
 $EndComp
 $Comp
-L big_battery-rescue:AP1117-ADJ-Regulator_Linear U1
+L Regulator_Linear:AP1117-ADJ U1
 U 1 1 5BCEBAD3
 P 3050 1000
@@
 $EndComp
 $Comp
-L big_battery-rescue:C_Small-Device C1
+L Device:C_Small C1
 U 1 1 5BCEBC6F
 P 2300 1200
@@
 $EndComp
 $Comp
-L big_battery-rescue:C_Small-Device C4
+L Device:C_Small C4
 U 1 1 5BCEBCFB
 P 3950 1200
@@
 $EndComp
 $Comp
-L big_battery-rescue:+12V-power #PWR03
+L power:+12V #PWR03
 U 1 1 5BCEBE59
 P 2300 850
@@
 	3950 1000 3950 1050
 $Comp
-L big_battery-rescue:R_Small-Device R7
+L Device:R_Small_US R7
 U 1 1 5BCEBF47
 P 3500 1200
@@
 $EndComp
 $Comp
-L big_battery-rescue:R_Small-Device R8
+L Device:R_Small_US R8
 U 1 1 5BCEC08F
 P 3500 1600
@@
 	3500 1000 3950 1000
 $Comp
-L big_battery-rescue:GND-power #PWR04
+L power:GND #PWR04
 U 1 1 5BCEC2C9
 P 2300 1750
@@
 $EndComp
 $Comp
-L big_battery-rescue:GND-power #PWR09
+L power:GND #PWR09
 U 1 1 5BCEC2F3
 P 3500 1750
@@
 $EndComp
 $Comp
-L big_battery-rescue:GND-power #PWR011
+L power:GND #PWR011
 U 1 1 5BCEC316
 P 3950 1750
@@
 	2300 1300 2300 1350
 $Comp
-L big_battery-rescue:+3V3-power #PWR010
+L power:+3.3V #PWR010
 U 1 1 5BCEC946
 P 3950 850
@@
 Connection ~ 3950 1000
 $Comp
-L big_battery-rescue:R_Small-Device R3
+L Device:R_Small_US R3
 U 1 1 5BCED0F5
 P 2300 5200
@@
 $EndComp
 $Comp
-L big_battery-rescue:R_Small-Device R4
+L Device:R_Small_US R4
 U 1 1 5BCED19D
 P 2650 4850
@@
 CB
 $Comp
-L big_battery-rescue:+3V3-power #PWR05
+L power:+3.3V #PWR05
 U 1 1 5BCEDDE7
 P 2650 4350
@@
 	3400 4450 3100 4450
 $Comp
-L big_battery-rescue:GND-power #PWR08
+L power:GND #PWR08
 U 1 1 5BCEE89B
 P 3400 4750
@@
 	3400 4700 3400 4750
 $Comp
-L big_battery-rescue:C_Small-Device C2
+L Device:C_Small C2
 U 1 1 5BCEFC9A
 P 3100 6500
@@
 $EndComp
 $Comp
-L big_battery-rescue:R_Small-Device R6
+L Device:R_Small_US R6
 U 1 1 5BCEFDEB
 P 3100 6150
@@
 $EndComp
 $Comp
-L big_battery-rescue:R_Small-Device R5
+L Device:R_Small_US R5
 U 1 1 5BCEFEBA
 P 2650 6750
@@
 $EndComp
 $Comp
-L big_battery-rescue:GND-power #PWR07
+L power:GND #PWR07
 U 1 1 5BCF04BA
 P 3100 5650
@@
 Connection ~ 2650 6500
 $Comp
-L big_battery-rescue:GND-power #PWR06
+L power:GND #PWR06
 U 1 1 5BCF396D
 P 2650 6950
@@
 	2650 4450 2650 4750
 $Comp
-L big_battery-rescue:R_Small-Device R14
+L Device:R_Small_US R14
 U 1 1 5BCFEDF2
 P 7350 4550
@@
 $EndComp
 $Comp
-L big_battery-rescue:C_Small-Device C5
+L Device:C_Small C5
 U 1 1 5BCFEF1E
 P 7000 4550
@@
 $EndComp
 $Comp
-L big_battery-rescue:R_Small-Device R13
+L Device:R_Small_US R13
 U 1 1 5BCFF056
 P 6550 5650
@@
 $EndComp
 $Comp
-L big_battery-rescue:R_Small-Device R11
+L Device:R_Small_US R11
 U 1 1 5BCFF18F
 P 5950 5650
@@
 $EndComp
 $Comp
-L big_battery-rescue:Q_NMOS_GSD-Device Q1
+L Device:Q_NMOS_GSD Q1
 U 1 1 5BCFF343
 P 5850 6050
@@
 $EndComp
 $Comp
-L big_battery-rescue:R_Small-Device R10
+L Device:R_Small_US R10
 U 1 1 5BCFF619
 P 5500 6250
@@
 $EndComp
 $Comp
-L big_battery-rescue:R_Small-Device R9
+L Device:R_Small_US R9
 U 1 1 5BCFF687
 P 5200 6050
@@
 $EndComp
 $Comp
-L big_battery-rescue:R_Small-Device R12
+L Device:R_Small_US R12
 U 1 1 5BCFF770
 P 6250 4450
@@
 	5950 6500 5950 6250
 $Comp
-L big_battery-rescue:GND-power #PWR015
+L power:GND #PWR015
 U 1 1 5BD08424
 P 6250 6650
@@
 	6250 6500 5950 6500
 $Comp
-L big_battery-rescue:+3V3-power #PWR014
+L power:+3.3V #PWR014
 U 1 1 5BD0D06A
 P 6250 4300
@@
 TRICKLE_DIS
 $Comp
-L big_battery-rescue:R_Small-Device R16
+L Device:R_Small_US R16
 U 1 1 5BD15B9A
 P 8750 5450
@@
 $EndComp
 $Comp
-L big_battery-rescue:R_Small-Device R15
+L Device:R_Small_US R15
 U 1 1 5BD15C2E
 P 8750 4850
@@
 	8750 4750 8750 4550
 $Comp
-L big_battery-rescue:GND-power #PWR017
+L power:GND #PWR017
 U 1 1 5BD20C57
 P 8750 5800
@@
 $EndComp
 $Comp
-L big_battery-rescue:+3V3-power #PWR016
+L power:+3.3V #PWR016
 U 1 1 5BD20D04
 P 8750 4550
@@
 	8750 4950 8750 5150
 $Comp
-L big_battery-rescue:D_Schottky_Small-Device D1
+L Device:D_Schottky_Small D1
 U 1 1 5BD1078D
 P 8000 5200
@@
 	8750 5200 8750 5350
 $Comp
-L big_battery-rescue:C_Small-Device C6
+L Device:C_Small C6
 U 1 1 5BD14EFB
 P 8350 5450
@@
 	2600 3200 2850 3200
 $Comp
-L big_battery-rescue:R_Small-Device R2
+L Device:R_Small_US R2
 U 1 1 5BD23F1D
 P 2250 3250
@@
 $EndComp
 $Comp
-L big_battery-rescue:R_Small-Device R1
+L Device:R_Small_US R1
 U 1 1 5BD23FA1
 P 2250 2750
@@
 HAD TO USE UP EXTRA OP-AMP
 $Comp
-L big_battery-rescue:GND-power #PWR02
+L power:GND #PWR02
 U 1 1 5BD28CB4
 P 2250 3550
@@
 V_Out
 $Comp
-L big_battery-rescue:Conn_01x02_Female-Connector J2
+L Connector:Conn_01x02_Female J2
 U 1 1 5BD0A582
 P 900 1150
@@
 	1400 4200 1400 5450
 $Comp
-L big_battery-rescue:GND-power #PWR01
+L power:GND #PWR01
 U 1 1 5BD41058
 P 1400 5450
@@
 	3550 5300 4800 5300
 $Comp
-L big_battery-rescue:Conn_01x04_Female-Connector J1
+L Connector:Conn_01x04_Female J1
 U 1 1 5BD54D73
 P 850 4000
@@
 Voltage Trim
 $Comp
-L big_battery-rescue:C_Small-Device C7
+L Device:C_Small C7
 U 1 1 5BCFF17E
 P 1900 3250
@@
 	4900 6050 5100 6050
 $Comp
-L big_battery-rescue:Conn_01x04_Female-Connector J3
+L Connector:Conn_01x04_Female J3
 U 1 1 5BD0CE4E
 P 10600 3200
@@
 $EndComp
 $Comp
-L big_battery-rescue:GND-power #PWR0101
+L power:GND #PWR0101
 U 1 1 5BD15DF3
 P 10250 3500
@@
 	5500 6050 5650 6050
 $Comp
-L big_battery-rescue:LED_Small-Device D2
+L Device:LED_Small D2
 U 1 1 5BD9A687
 P 4450 1500
@@
 $EndComp
 $Comp
-L big_battery-rescue:R_Small-Device R17
+L Device:R_Small_US R17
 U 1 1 5BD9AD09
 P 4450 1250

Commit message: adds big battery v2.0
Parts:
- R1, R10, R11, R12, R13, R14, R15, R16, R17, R2, R3, R4, R5, R6, R7, R8, R9: symbol Device:R_Small_US -> Device:R_Small
Changed lines of the file:
@@
 	3950 1000 3950 1050
 $Comp
-L Device:R_Small_US R7
+L Device:R_Small R7
 U 1 1 5BCEBF47
 P 3500 1200
@@
 $EndComp
 $Comp
-L Device:R_Small_US R8
+L Device:R_Small R8
 U 1 1 5BCEC08F
 P 3500 1600
@@
 Connection ~ 3950 1000
 $Comp
-L Device:R_Small_US R3
+L Device:R_Small R3
 U 1 1 5BCED0F5
 P 2300 5200
@@
 $EndComp
 $Comp
-L Device:R_Small_US R4
+L Device:R_Small R4
 U 1 1 5BCED19D
 P 2650 4850
@@
 $EndComp
 $Comp
-L Device:R_Small_US R6
+L Device:R_Small R6
 U 1 1 5BCEFDEB
 P 3100 6150
@@
 $EndComp
 $Comp
-L Device:R_Small_US R5
+L Device:R_Small R5
 U 1 1 5BCEFEBA
 P 2650 6750
@@
 	2650 4450 2650 4750
 $Comp
-L Device:R_Small_US R14
+L Device:R_Small R14
 U 1 1 5BCFEDF2
 P 7350 4550
@@
 $EndComp
 $Comp
-L Device:R_Small_US R13
+L Device:R_Small R13
 U 1 1 5BCFF056
 P 6550 5650
@@
 $EndComp
 $Comp
-L Device:R_Small_US R11
+L Device:R_Small R11
 U 1 1 5BCFF18F
 P 5950 5650
@@
 $EndComp
 $Comp
-L Device:R_Small_US R10
+L Device:R_Small R10
 U 1 1 5BCFF619
 P 5500 6250
@@
 $EndComp
 $Comp
-L Device:R_Small_US R9
+L Device:R_Small R9
 U 1 1 5BCFF687
 P 5200 6050
@@
 $EndComp
 $Comp
-L Device:R_Small_US R12
+L Device:R_Small R12
 U 1 1 5BCFF770
 P 6250 4450
@@
 TRICKLE_DIS
 $Comp
-L Device:R_Small_US R16
+L Device:R_Small R16
 U 1 1 5BD15B9A
 P 8750 5450
@@
 $EndComp
 $Comp
-L Device:R_Small_US R15
+L Device:R_Small R15
 U 1 1 5BD15C2E
 P 8750 4850
@@
 	2600 3200 2850 3200
 $Comp
-L Device:R_Small_US R2
+L Device:R_Small R2
 U 1 1 5BD23F1D
 P 2250 3250
@@
 $EndComp
 $Comp
-L Device:R_Small_US R1
+L Device:R_Small R1
 U 1 1 5BD23FA1
 P 2250 2750
@@
 $EndComp
 $Comp
-L Device:R_Small_US R17
+L Device:R_Small R17
 U 1 1 5BD9AD09
 P 4450 1250
