File: kicad/big_battery_v2.0/big_battery.kicad_pcb (KiCad board)
At the start: 2 copper layers, 75 x 45 mm, 86 parts, among them J1 CN3, J2 CN2, J3 MCU, J4 P1, J5 P0, J6 PRGM, J7 DI, J8 DO, Q1 AO3400, Q2 AO3400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

Commit message: fixing up silkscreen
Parts:
- RV1: value R_POT -> TRK_ADJ
- RV2: value R_POT -> I_ADJ
- RV3: value R_POT -> V_ADJ
- moved JP2 6.00 mm to (47.6, 28.0)
- moved JP4 6.00 mm to (47.6, 34.0)
- moved L4 5.89 mm to (54.5, 32.1), turned to 270 degrees
- moved C10 4.37 mm to (56.5, 32.1), turned to 90 degrees
- moved U4 3.60 mm to (60.6, 32.1)
- turned C11 to 180 degrees
- turned JP8 to 180 degrees
- turned R22 to 180 degrees
- turned R26 to 180 degrees
Connections:
- net Net-(D3-Pad1) renamed /I_LIMIT
- net Net-(J7-Pad1) renamed /DI_ANODE
- net Net-(J7-Pad2) renamed /DI_CATHODE
- net Net-(J8-Pad1) renamed /DO_EMITTER
- net Net-(J8-Pad2) renamed /DO_COLLECTOR
- net Net-(JP10-Pad1) renamed /V_PWM
- net Net-(JP8-Pad1) renamed /I_PWM
- net Net-(Q3-Pad3) renamed /DO_CATHODE
- net Net-(R31-Pad1) renamed /DO_ANODE
Routing:
- net /VOLTAGE: track 0.00 -> 81.3 mm, vias 0 -> 4
- net Net-(C6-Pad1): track 0.00 -> 63.1 mm, vias 0 -> 2
- net /P0.1: track 0.00 -> 44.9 mm, vias 0 -> 3
- net /P0.7: track 0.00 -> 43.7 mm
- net /P0.2: track 0.00 -> 43.7 mm, vias 0 -> 3
- net /P0.5: track 0.00 -> 43.5 mm, vias 0 -> 2
- net /P0.0: track 0.00 -> 40.9 mm, vias 0 -> 1
- net /P0.3: track 0.00 -> 39.9 mm, vias 0 -> 1
- net /CURRENT: track 47.6 -> 86.9 mm, vias 0 -> 4
- net /P0.4: track 0.00 -> 36.0 mm, vias 0 -> 1
- net /TRICKLE_DIS: track 15.7 -> 49.9 mm, vias 0 -> 2
- net Net-(C5-Pad2): track 13.7 -> 46.7 mm, vias 0 -> 3
- net /P0.6: track 0.00 -> 19.6 mm
- net Net-(D1-Pad1): track 2.93 -> 22.2 mm, vias 0 -> 4
- net Net-(Q3-Pad1): track 0.00 -> 18.7 mm
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Other:
- net class Default: clearance 0.4 -> 0.2
- rule trace_clearance: 0.4 -> 0.2
- board text added: "12V"
- board text added: "3V3"
- board text added: "C2CK"
- board text added: "C2D"
- board text added: "CB"
- board text added: "CURRENT"
- board text added: "CURR_PWM"
- board text added: "DI_AN"
- board text added: "DI_CAT"
- board text added: "DO_COLLECTOR"
- board text added: "DO_EMITTER"
- board text added: "GND"
- board text added: "I_ADJ"
- board text added: "I_LIMIT"
- board text added: "I_PWM"
- board text added: "P0.0"
- board text added: "P0.1"
- board text added: "P0.2"
- board text added: "P0.3"
- board text added: "P0.4"
- board text added: "P0.5"
- board text added: "P0.6"
- board text added: "P0.7"
- board text added: "P1.0"
- board text added: "P1.1"
- board text added: "P1.2"
- board text added: "P1.3"
- board text added: "P1.4"
- board text added: "P1.5"
- board text added: "P1.6"
- board text added: "RC1"
- board text added: "RCG"
- board text added: "S+"
- board text added: "TRICKLE_DIS"
- board text added: "TRK_ADJ"
- board text added: "TRM"
- board text added: "VOLTAGE"
- board text added: "VOLT_PWM"
- board text added: "V_ADJ"
- board text added: "V_PWM"
- board text added: "~OUTPUT_EN"

Commit message: final gerbers sent out
Parts:
- added G***: LOGO, logo:logo_large, B.Cu at (57.0, 32.5)
- added J9: PWM, Connector_JST:JST_EH_B02B-EH-A_1x02_P2.50mm_Vertical, F.Cu at (39.9, 42.0)
- moved RV3 3.85 mm to (34.2, 42.0)
- moved RV1 3.26 mm to (23.8, 42.0)
- moved RV2 2.65 mm to (13.4, 42.0)
- moved J6 1.77 mm to (48.7, 42.0)
Routing:
- net /VOLTAGE_PWM: track 13.2 -> 39.2 mm, vias 0 -> 2
- net /CURRENT_PWM: track 7.54 -> 24.8 mm, vias 0 -> 2
- net +3V3: track 244.9 -> 236.9 mm
- net Net-(C6-Pad1): track 63.1 -> 67.2 mm
- net /P0.2: track 43.7 -> 47.3 mm
- net /P0.3: track 39.9 -> 43.5 mm
- net Net-(R16-Pad1): track 6.38 -> 9.77 mm
- net Net-(R13-Pad1): track 5.60 -> 7.18 mm
- net /P0.0: track 40.9 -> 39.4 mm
- net /P0.1: track 44.9 -> 43.7 mm
- net /VOLTAGE: track 81.3 -> 82.4 mm
- net /CURRENT: track 86.9 -> 87.8 mm
- net /C2CK: track 13.4 -> 12.6 mm
- net Net-(R11-Pad2): track 5.68 -> 6.36 mm
- net GND: vias 41 -> 37
Other:
- board text added: "BIG_BATT V2.0 181120 FITZ"
- board text added: "DI"
- board text added: "DO"
