File: kicad/big_battery_v2.0/big_battery.sch (KiCad schematic (older format))
At the start: 86 parts, among them J1 CN3, J2 CN2, J3 MCU, J4 P1, J5 P0, J6 PRGM, J7 DI, J8 DO, Q1 AO3400, Q2 AO3400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

Commit message: fixing up silkscreen
Parts:
- RV1: value R_POT -> TRK_ADJ
- RV2: value R_POT -> I_ADJ
- RV3: value R_POT -> V_ADJ
Connections:
- net V_PWM: now reaches JP10.1, R27.2, U3.7
- net I_PWM: now reaches JP8.1, R23.2, U3.1
- net DI_ANODE: now reaches J7.1 (Pin_1), U5.1
- net DI_CATHODE: now reaches J7.2 (Pin_2), U5.2
- net I_LIMIT: now reaches D3.1 (K), JP9.2
- net DO_CATHODE: now reaches Q3.3 (D), U6.2
- net DO_EMITTER: now reaches J8.1 (Pin_1), U6.3
- net DO_COLLECTOR: now reaches J8.2 (Pin_2), U6.4
- net DO_ANODE: now reaches R31.1, U6.1
Changed lines of the file:
@@
 P 5500 9400
 F 0 "RV1" H 5430 9446 50  0000 R CNN
-F 1 "R_POT" H 5430 9355 50  0000 R CNN
+F 1 "TRK_ADJ" H 5430 9355 50  0000 R CNN
 F 2 "Potentiometer_THT:Potentiometer_Bourns_3296W_Vertical" H 5500 9400 50  0001 C CNN
 F 3 "~" H 5500 9400 50  0001 C CNN
@@
 P 6100 9400
 F 0 "RV2" H 6030 9446 50  0000 R CNN
-F 1 "R_POT" H 6030 9355 50  0000 R CNN
+F 1 "I_ADJ" H 6030 9355 50  0000 R CNN
 F 2 "Potentiometer_THT:Potentiometer_Bourns_3296W_Vertical" H 6100 9400 50  0001 C CNN
 F 3 "~" H 6100 9400 50  0001 C CNN
@@
 P 8800 9200
 F 0 "RV3" H 8730 9246 50  0000 R CNN
-F 1 "R_POT" H 8730 9155 50  0000 R CNN
+F 1 "V_ADJ" H 8730 9155 50  0000 R CNN
 F 2 "Potentiometer_THT:Potentiometer_Bourns_3296W_Vertical" H 8800 9200 50  0001 C CNN
 F 3 "~" H 8800 9200 50  0001 C CNN
@@
 Wire Wire Line
 	9200 2900 9200 3050
+Text Label 8950 4700 0    50   ~ 0
+V_PWM
+Text Label 6350 4700 0    50   ~ 0
+I_PWM
+Text Label 9200 3050 2    50   ~ 0
+DO_ANODE
+Text Label 9200 3250 2    50   ~ 0
+DO_CATHODE
+Text Label 10100 3050 0    50   ~ 0
+DO_COLLECTOR
+Text Label 10100 3250 0    50   ~ 0
+DO_EMITTER
+Text Label 1900 2650 0    50   ~ 0
+DI_ANODE
+Text Label 1900 2750 0    50   ~ 0
+DI_CATHODE
+Text Label 3000 2650 0    50   ~ 0
+DI_COLLECTOR
+Text Label 3000 2850 0    50   ~ 0
+DI_EMITTER
+Text Label 7850 8400 0    50   ~ 0
+I_LIMIT
 $EndSCHEMATC

Commit message: final gerbers sent out
Parts:
- added J9: PWM, Connector_JST:JST_EH_B02B-EH-A_1x02_P2.50mm_Vertical, symbol Connector_Generic:Conn_01x02
Connections:
- net CURRENT_PWM: now also J9.1 (Pin_1)
- net VOLTAGE_PWM: now also J9.2 (Pin_2)
Other:
- moved on the sheet: Q2, R18, R19
Changed lines of the file:
@@
 Connection ~ 4150 6250
 Wire Wire Line
-	4250 2350 4250 4600
+	4250 2350 4250 3550
 Wire Wire Line
 	4250 4600 4500 4600
 Wire Wire Line
-	4350 2450 4350 3700
-Wire Wire Line
-	4350 3700 6950 3700
-Wire Wire Line
-	6950 3700 6950 4600
+	4350 2450 4350 3650
+Wire Wire Line
+	4350 3650 6950 3650
+Wire Wire Line
+	6950 3650 6950 4600
 Wire Wire Line
 	6800 4700 6800 8850
@@
 L big_battery-rescue:Q_NMOS_GSD-Device Q2
 U 1 1 5C8B7C86
-P 2050 4250
-F 0 "Q2" H 2255 4296 50  0000 L CNN
-F 1 "AO3400" H 2255 4205 50  0000 L CNN
-F 2 "Package_TO_SOT_SMD:SOT-23_Handsoldering" H 2250 4350 50  0001 C CNN
-F 3 "~" H 2050 4250 50  0001 C CNN
-	1    2050 4250
+P 2050 4600
+F 0 "Q2" H 2255 4646 50  0000 L CNN
+F 1 "AO3400" H 2255 4555 50  0000 L CNN
+F 2 "Package_TO_SOT_SMD:SOT-23_Handsoldering" H 2250 4700 50  0001 C CNN
+F 3 "~" H 2050 4600 50  0001 C CNN
+	1    2050 4600
 	-1   0    0    -1
 $EndComp
@@
 	1350 1350 1350 6650
 Wire Wire Line
-	1450 3850 1950 3850
-Wire Wire Line
-	1950 3850 1950 4050
-Wire Wire Line
-	1450 3850 1450 6750
+	1450 4200 1950 4200
+Wire Wire Line
+	1950 4200 1950 4400
+Wire Wire Line
+	1450 4200 1450 6750
 $Comp
 L big_battery-rescue:R_Small-Device R19
 U 1 1 5C91C427
-P 2600 4250
-F 0 "R19" V 2796 4250 50  0000 C CNN
-F 1 "1K" V 2705 4250 50  0000 C CNN
-F 2 "Resistor_SMD:R_0603_1608Metric_Pad1.05x0.95mm_HandSolder" H 2600 4250 50  0001 C CNN
-F 3 "~" H 2600 4250 50  0001 C CNN
-	1    2600 4250
+P 2600 4600
+F 0 "R19" V 2796 4600 50  0000 C CNN
+F 1 "1K" V 2705 4600 50  0000 C CNN
+F 2 "Resistor_SMD:R_0603_1608Metric_Pad1.05x0.95mm_HandSolder" H 2600 4600 50  0001 C CNN
+F 3 "~" H 2600 4600 50  0001 C CNN
+	1    2600 4600
 	0    -1   -1   0
 $EndComp
@@
 L big_battery-rescue:R_Small-Device R18
 U 1 1 5C91C717
-P 2350 3900
-F 0 "R18" H 2291 3854 50  0000 R CNN
-F 1 "100K" H 2291 3945 50  0000 R CNN
-F 2 "Resistor_SMD:R_0603_1608Metric_Pad1.05x0.95mm_HandSolder" H 2350 3900 50  0001 C CNN
-F 3 "~" H 2350 3900 50  0001 C CNN
-	1    2350 3900
+P 2350 4250
+F 0 "R18" H 2291 4204 50  0000 R CNN
+F 1 "100K" H 2291 4295 50  0000 R CNN
+F 2 "Resistor_SMD:R_0603_1608Metric_Pad1.05x0.95mm_HandSolder" H 2350 4250 50  0001 C CNN
+F 3 "~" H 2350 4250 50  0001 C CNN
+	1    2350 4250
 	1    0    0    1
 $EndComp
@@
 L big_battery-rescue:GND-power #PWR0120
 U 1 1 5C9461A6
-P 1950 4800
-F 0 "#PWR0120" H 1950 4550 50  0001 C CNN
-F 1 "GND" H 1955 4627 50  0000 C CNN
-F 2 "" H 1950 4800 50  0001 C CNN
-F 3 "" H 1950 4800 50  0001 C CNN
-	1    1950 4800
-	1    0    0    -1
-$EndComp
-Wire Wire Line
-	2250 4250 2350 4250
-Wire Wire Line
-	1950 4450 1950 4800
+P 1950 5050
+F 0 "#PWR0120" H 1950 4800 50  0001 C CNN
+F 1 "GND" H 1955 4877 50  0000 C CNN
+F 2 "" H 1950 5050 50  0001 C CNN
+F 3 "" H 1950 5050 50  0001 C CNN
+	1    1950 5050
+	1    0    0    -1
+$EndComp
+Wire Wire Line
+	2250 4600 2350 4600
+Wire Wire Line
+	1950 4800 1950 5050
 $Comp
 L big_battery-rescue:+3V3-power #PWR0121
 U 1 1 5C971343
-P 2350 3700
-F 0 "#PWR0121" H 2350 3550 50  0001 C CNN
-F 1 "+3V3" H 2365 3873 50  0000 C CNN
-F 2 "" H 2350 3700 50  0001 C CNN
-F 3 "" H 2350 3700 50  0001 C CNN
-	1    2350 3700
-	1    0    0    -1
-$EndComp
-Wire Wire Line
-	2350 3700 2350 3800
-Wire Wire Line
-	2350 4000 2350 4250
-Connection ~ 2350 4250
-Wire Wire Line
-	2350 4250 2500 4250
+P 2350 4050
+F 0 "#PWR0121" H 2350 3900 50  0001 C CNN
+F 1 "+3V3" H 2365 4223 50  0000 C CNN
+F 2 "" H 2350 4050 50  0001 C CNN
+F 3 "" H 2350 4050 50  0001 C CNN
+	1    2350 4050
+	1    0    0    -1
+$EndComp
+Wire Wire Line
+	2350 4050 2350 4150
+Wire Wire Line
+	2350 4350 2350 4600
+Connection ~ 2350 4600
+Wire Wire Line
+	2350 4600 2500 4600
 $Comp
 L Device:Jumper_NO_Small JP7
@@
 	5450 2550 6350 2550
 Wire Wire Line
-	3850 4250 3850 2550
-Wire Wire Line
-	2700 4250 3850 4250
+	3850 4600 3850 2550
+Wire Wire Line
+	2700 4600 3850 4600
 Wire Wire Line
 	3850 2550 5250 2550
@@
 	1    0    0    -1
 $EndComp
-Text Label 1950 4700 0    50   ~ 0
+Text Label 1950 4950 0    50   ~ 0
 AUXG
-Text Label 1950 3850 0    50   ~ 0
+Text Label 1950 4200 0    50   ~ 0
 RCG
 $Comp
@@
 Text Notes 2250 2350 0    50   ~ 0
 ISOLATED DATA IN
-Text Notes 1600 3650 0    50   ~ 0
+Text Notes 1600 4000 0    50   ~ 0
 REMOTE ON/OFF
 Text Notes 1600 6550 0    50   ~ 0
@@
 Text Label 7850 8400 0    50   ~ 0
 I_LIMIT
+$Comp
+L Connector_Generic:Conn_01x02 J9
+U 1 1 5C4891A7
+P 1700 3550
+F 0 "J9" H 1620 3767 50  0000 C CNN
+F 1 "PWM" H 1620 3676 50  0000 C CNN
+F 2 "Connector_JST:JST_EH_B02B-EH-A_1x02_P2.50mm_Vertical" H 1700 3550 50  0001 C CNN
+F 3 "~" H 1700 3550 50  0001 C CNN
+	1    1700 3550
+	-1   0    0    -1
+$EndComp
+Wire Wire Line
+	4350 3650 1900 3650
+Connection ~ 4350 3650
+Wire Wire Line
+	4250 3550 1900 3550
+Connection ~ 4250 3550
+Wire Wire Line
+	4250 3550 4250 4600
 $EndSCHEMATC

Commit message: adds first firmware version
Parts:
- R11: value 18K 1% -> 0R
- R13: value 10K 1% -> 0R
- R16: value 12K 1% -> 0R
- R22, R26: value 1R -> NC
- R23, R27: value 1R -> 0R
- RV1: value TRK_ADJ -> 50K
- RV2: value I_ADJ -> 50K
- RV3: value V_ADJ -> 50K
Changed lines of the file:
@@
 P 6100 9850
 F 0 "R13" H 6041 9896 50  0000 R CNN
-F 1 "10K 1%" H 6041 9805 50  0000 R CNN
+F 1 "0R" H 6041 9805 50  0000 R CNN
 F 2 "Resistor_SMD:R_0603_1608Metric_Pad1.05x0.95mm_HandSolder" H 6100 9850 50  0001 C CNN
 F 3 "~" H 6100 9850 50  0001 C CNN
@@
 P 5500 9850
 F 0 "R11" H 5441 9804 50  0000 R CNN
-F 1 "18K 1%" H 5441 9895 50  0000 R CNN
+F 1 "0R" H 5441 9895 50  0000 R CNN
 F 2 "Resistor_SMD:R_0603_1608Metric_Pad1.05x0.95mm_HandSolder" H 5500 9850 50  0001 C CNN
 F 3 "~" H 5500 9850 50  0001 C CNN
@@
 P 8800 9650
 F 0 "R16" H 8741 9696 50  0000 R CNN
-F 1 "12K 1%" H 8741 9605 50  0000 R CNN
+F 1 "0R" H 8741 9605 50  0000 R CNN
 F 2 "Resistor_SMD:R_0603_1608Metric_Pad1.05x0.95mm_HandSolder" H 8800 9650 50  0001 C CNN
 F 3 "~" H 8800 9650 50  0001 C CNN
@@
 P 5500 9400
 F 0 "RV1" H 5430 9446 50  0000 R CNN
-F 1 "TRK_ADJ" H 5430 9355 50  0000 R CNN
+F 1 "50K" H 5430 9355 50  0000 R CNN
 F 2 "Potentiometer_THT:Potentiometer_Bourns_3296W_Vertical" H 5500 9400 50  0001 C CNN
 F 3 "~" H 5500 9400 50  0001 C CNN
@@
 P 6100 9400
 F 0 "RV2" H 6030 9446 50  0000 R CNN
-F 1 "I_ADJ" H 6030 9355 50  0000 R CNN
+F 1 "50K" H 6030 9355 50  0000 R CNN
 F 2 "Potentiometer_THT:Potentiometer_Bourns_3296W_Vertical" H 6100 9400 50  0001 C CNN
 F 3 "~" H 6100 9400 50  0001 C CNN
@@
 P 8800 9200
 F 0 "RV3" H 8730 9246 50  0000 R CNN
-F 1 "V_ADJ" H 8730 9155 50  0000 R CNN
+F 1 "50K" H 8730 9155 50  0000 R CNN
 F 2 "Potentiometer_THT:Potentiometer_Bourns_3296W_Vertical" H 8800 9200 50  0001 C CNN
 F 3 "~" H 8800 9200 50  0001 C CNN
@@
 P 6300 5300
 F 0 "R23" V 6496 5300 50  0000 C CNN
-F 1 "1R" V 6405 5300 50  0000 C CNN
+F 1 "0R" V 6405 5300 50  0000 C CNN
 F 2 "Resistor_SMD:R_0603_1608Metric_Pad1.05x0.95mm_HandSolder" H 6300 5300 50  0001 C CNN
 F 3 "~" H 6300 5300 50  0001 C CNN
@@
 P 5600 5450
 F 0 "R22" V 5796 5450 50  0000 C CNN
-F 1 "1R" V 5705 5450 50  0000 C CNN
+F 1 "NC" V 5705 5450 50  0000 C CNN
 F 2 "Resistor_SMD:R_0603_1608Metric_Pad1.05x0.95mm_HandSolder" H 5600 5450 50  0001 C CNN
 F 3 "~" H 5600 5450 50  0001 C CNN
@@
 P 8900 5300
 F 0 "R27" V 9096 5300 50  0000 C CNN
-F 1 "1R" V 9005 5300 50  0000 C CNN
+F 1 "0R" V 9005 5300 50  0000 C CNN
 F 2 "Resistor_SMD:R_0603_1608Metric_Pad1.05x0.95mm_HandSolder" H 8900 5300 50  0001 C CNN
 F 3 "~" H 8900 5300 50  0001 C CNN
@@
 P 8200 5450
 F 0 "R26" V 8396 5450 50  0000 C CNN
-F 1 "1R" V 8305 5450 50  0000 C CNN
+F 1 "NC" V 8305 5450 50  0000 C CNN
 F 2 "Resistor_SMD:R_0603_1608Metric_Pad1.05x0.95mm_HandSolder" H 8200 5450 50  0001 C CNN
 F 3 "~" H 8200 5450 50  0001 C CNN

Commit message: got gpio working
Other:
- note added: "DI/DO and VOLTAGE_PWM/OUTPUT_EN are switched respectively"
- note added: "DI/DO must be on P0.4/ P0.5"
Changed lines of the file:
@@
 Wire Wire Line
 	4250 3550 4250 4600
+Text Notes 3900 2900 0    50   ~ 0
+DI/DO and VOLTAGE_PWM/OUTPUT_EN are switched respectively
+Text Notes 5000 3000 0    50   ~ 0
+DI/DO must be on P0.4/ P0.5
 $EndSCHEMATC

Commit message: updated schematic to include bodge wires
Parts:
- R28: value 10K 1% -> 1K %1
- R31: value 10K 1% -> 1K 1%
Other:
- note added: "BODGE WIRE"
- note added: "LEAVE UNPLACED\n"
Changed lines of the file:
@@
 P 3150 2450
 F 0 "R28" H 3091 2404 50  0000 R CNN
-F 1 "10K 1%" H 3091 2495 50  0000 R CNN
+F 1 "1K %1" H 3091 2495 50  0000 R CNN
 F 2 "Resistor_SMD:R_0603_1608Metric_Pad1.05x0.95mm_HandSolder" H 3150 2450 50  0001 C CNN
 F 3 "~" H 3150 2450 50  0001 C CNN
@@
 P 9200 2800
 F 0 "R31" H 9141 2754 50  0000 R CNN
-F 1 "10K 1%" H 9141 2845 50  0000 R CNN
+F 1 "1K 1%" H 9141 2845 50  0000 R CNN
 F 2 "Resistor_SMD:R_0603_1608Metric_Pad1.05x0.95mm_HandSolder" H 9200 2800 50  0001 C CNN
 F 3 "~" H 9200 2800 50  0001 C CNN
@@
 Text Notes 5000 3000 0    50   ~ 0
 DI/DO must be on P0.4/ P0.5
+Wire Notes Line
+	8300 3300 8300 3950
+Wire Notes Line
+	8300 3950 9500 3950
+Wire Notes Line
+	9500 3950 9500 3300
+Wire Notes Line
+	9500 3300 8300 3300
+Text Notes 9700 3850 0    50   ~ 0
+LEAVE UNPLACED\n
+Wire Bus Line
+	9200 3250 8000 3250
+Wire Bus Line
+	8000 3250 8000 3550
+Text Notes 8000 3250 0    50   ~ 0
+BODGE WIRE
+Wire Bus Line
+	5500 2450 5500 2600
+Wire Bus Line
+	5500 2600 5200 2600
+Wire Bus Line
+	5200 2600 5200 2650
+Wire Bus Line
+	5200 2750 5200 2700
+Wire Bus Line
+	5200 2700 5600 2700
+Wire Bus Line
+	5600 2700 5600 2550
+Wire Bus Line
+	5150 2450 5150 2800
+Wire Bus Line
+	5150 2800 5700 2800
+Wire Bus Line
+	5700 2800 5700 2650
+Wire Bus Line
+	5050 2550 5050 2900
+Wire Bus Line
+	5050 2900 5800 2900
+Wire Bus Line
+	5800 2900 5800 2750
 $EndSCHEMATC
