File: kicad/big_battery_v3/big_battery_v3.sch (KiCad schematic (older format))
At the start: 88 parts, among them J1 CN3, J2 CN2, J3 MCU, J4 P1, J5 P0, J6 PRGM, J7 DI, J8 DO, J9 PWM, Q1 AO3400, Q2 AO3400, Q3 AO3400, U1 AP1117-ADJ, U2 LMV324, U3 LMV358, U4 EFM8BB10F2G-A-QFN20, U5 PC817, U6 PC817

Commit message: adds big battery v3
Parts:
- removed Q3: AO3400, Package_TO_SOT_SMD:SOT-23_Handsoldering, symbol big_battery-rescue:Q_NMOS_GSD-Device
- removed R29: 1K, Resistor_SMD:R_0603_1608Metric_Pad1.05x0.95mm_HandSolder, symbol big_battery-rescue:R_Small-Device
- removed R30: 100K, Resistor_SMD:R_0603_1608Metric_Pad1.05x0.95mm_HandSolder, symbol big_battery-rescue:R_Small-Device
- C1, C10, C11, C2, C3, C4, C5, C6, C7, C8, C9: symbol big_battery-rescue:C_Small-Device -> Device:C_Small
- D1: footprint Diode_SMD:D_0603_1608Metric_Castellated -> Diode_SMD:D_SOD-323_HandSoldering; symbol big_battery-rescue:D_Schottky_Small-Device -> Device:D_Schottky
- D2, D3: symbol big_battery-rescue:LED_Small-Device -> Device:LED_Small
- J1: value CN3 -> CONN
- J3: value MCU -> CONN; symbol big_battery-rescue:Conn_01x04_Female-Connector -> Connector_Generic:Conn_01x04
- J6: value PRGM -> CONN
- J7: value DI -> CONN
- J8: value DO -> CONN
- J9: value PWM -> CONN
- L1, L2, L5: symbol big_battery-rescue:L_Small-Device -> Device:L_Small
- Q1, Q2: symbol big_battery-rescue:Q_NMOS_GSD-Device -> Device:Q_NMOS_GSD
- R1, R10, R11, R12, R13, R14, R15, R16, R17, R18, R19, R2, R20, R21, R22, R23, R24, R26, R27, R28, R3, R31, R32, R4, R5, R6, R7, R8, R9: symbol big_battery-rescue:R_Small-Device -> Device:R_Small
- R25: value 100K -> 10K; symbol big_battery-rescue:R_Small-Device -> Device:R_Small
- U1: symbol big_battery-rescue:AP1117-ADJ-Regulator_Linear -> Regulator_Linear:AP1117-ADJ
- U2: symbol big_battery-rescue:LMV324-Amplifier_Operational -> Amplifier_Operational:LMV324
Connections:
- wire segments 320 -> 315
Other:
- note added: "CN3"
- note added: "DI"
- note added: "MCU"
- note added: "PRGM\n"
- note added: "PWM"
- note removed: "BODGE WIRE"
- note removed: "DI/DO and VOLTAGE_PWM/OUTPUT_EN are switched respectively"
- note removed: "DI/DO must be on P0.4/ P0.5"
- note removed: "LEAVE UNPLACED\n"
